Commit message: se agrego un LIDAR pero no esta detectando

File: urdf/m2wr.urdf (robot description, URDF)
Before this commit: robot tortoisebot, 5 links, 4 joints
Links:
- added link hokuyo_link, mass 1e-5; collision box size=0.1 0.1 0.1; visual box size=0.1 0.1 0.1
Joints:
- added joint hokuyo_joint: type fixed, parent base_link, child hokuyo_link, origin xyz=0 0 0.2 rpy=0 0 0, axis 0 1 0
- joint front_caster_joint: origin xyz=0.3 0 0 rpy=0 0 0 -> xyz=0.25 0 0.009 rpy=0 0 0
